File: greatfet-one/greatfet-one.sch (KiCad schematic (older format))
At the start: 103 parts, among them J1 NEIGHBOR1, J2 NEIGHBOR2, J3 USB-MICRO-B-SHIELDED, J4 USB-MICRO-B-SHIELDED, J5 JTAG, J6 POWER, J7 BONUS_ROW, SW1 DFU, SW2 RESET, U1 LPC4330FBD144, U2 W25Q16DV, U3 AP7333, U4 IP4220CZ6, U5 AP2553W6-7, X1 MCU_XTAL, X2 RTC_XTAL

Commit message: GreatFET One: removed requirement for low insertion force headers for J1 and J2 now that we have the wiggler
Parts:
- J1, J2: Part Number SSW-120-21-L-D -> SSW-120-01-F-D
Changed lines of the file:
@@
 F 3 "" H 15750 1700 60  0000 C CNN
 F 4 "Samtec" H 15750 2650 60  0001 C CNN "Manufacturer"
-F 5 "SSW-120-21-L-D" H 15750 2650 60  0001 C CNN "Part Number"
+F 5 "SSW-120-01-F-D" H 15750 2650 60  0001 C CNN "Part Number"
 F 6 "CONN RCPT .100\" 40POS DUAL-ROW GOLD" H 15750 2650 60  0001 C CNN "Description"
 	1    15750 2650
@@
 F 3 "" H 15750 4300 60  0000 C CNN
 F 4 "Samtec" H 15750 5250 60  0001 C CNN "Manufacturer"
-F 5 "SSW-120-21-L-D" H 15750 5250 60  0001 C CNN "Part Number"
+F 5 "SSW-120-01-F-D" H 15750 5250 60  0001 C CNN "Part Number"
 F 6 "CONN RCPT .100\" 40POS DUAL-ROW GOLD" H 15750 5250 60  0001 C CNN "Description"
 	1    15750 5250

Commit message: GreatFET One: revised component selection based on availability
Parts:
- C1, C2, C5, C6, C8, C9: Manufacturer Murata -> Kemet; Part Number GRM1885C1H180JA01D -> C0603C180J5GAC
- C11, C4: Manufacturer Murata -> Taiyo Yuden; Part Number GRM21BR61A106KE19L -> LMK212ABJ106KG-T
- C12, C13, C14, C15, C16, C17, C18, C19, C20, C21, C22, C23, C24, C25, C7: Description CAP CER 0.1UF 16V 10% X7R 0603 -> CAP CER 0.1UF 16V 20% X7R 0603; Manufacturer Murata -> Kemet; Part Number GRM188R71C104KA01D -> C0603C104M4RAC
- J7: Manufacturer Samtec -> Sullins; Part Number TSW-120-07-L-S -> PRPC020SAAN-RC
- R19, R20: Manufacturer Rohm -> Yageo; Part Number MCR03ERTF33R0 -> RC0603FR-0733RL
