File: orchid/orchid.kicad_pcb (KiCad board)
At the start: 4 copper layers, 70.7 x 53.3 mm, 7 parts, among them J1 NEIGHBOR1, J2 NEIGHBOR2, J7 BONUS_ROW

Commit message: Working on Orchid pcb layout
Parts:
- added C1: 100pF, gsg-modules:0402, F.Cu at (138.4, 88.1)
- added C10: 220nF, gsg-modules:0402, F.Cu at (144.8, 87.9)
- added C11: 220nF, gsg-modules:0402, F.Cu at (146.8, 86.9)
- added C12: 200nF, gsg-modules:0402, F.Cu at (166.6, 80.5)
- added C13: 220nF, gsg-modules:0402, F.Cu at (154.2, 80.0)
- added C14: 220nF, gsg-modules:0402, F.Cu at (152.1, 81.0)
- added C15: 27pF, gsg-modules:0402, F.Cu at (132.6, 84.8)
- added C16: 27pF, gsg-modules:0402, F.Cu at (144.8, 86.9)
- added C17: 27pF, gsg-modules:0402, F.Cu at (146.8, 85.9)
- added C18: 27pF, gsg-modules:0402, F.Cu at (166.6, 81.5)
- added C19: 27pF, gsg-modules:0402, F.Cu at (154.2, 81.0)
- added C2: 100pF, gsg-modules:0402, F.Cu at (159.8, 78.7)
- added C20: 27pF, gsg-modules:0402, F.Cu at (152.1, 82.0)
- added C21: 18pF, gsg-modules:0402, F.Cu at (146.8, 84.8)
- added C22: 18pF, gsg-modules:0402, F.Cu at (152.1, 83.1)
- added C23: 1nF, gsg-modules:0402, F.Cu at (135.1, 82.5)
- added C24: 220nF, gsg-modules:0402, F.Cu at (144.9, 78.9)
- added C25: 1nF, gsg-modules:0402, F.Cu at (163.8, 84.3)
- added C26: 220nF, gsg-modules:0402, F.Cu at (153.2, 89.2)
- added C27: 27pF, gsg-modules:0402, F.Cu at (143.9, 78.9)
- added C28: 18pF, gsg-modules:0402, F.Cu at (146.8, 83.3)
- added C29: 27pF, gsg-modules:0402, F.Cu at (154.2, 89.2)
- added C3: 220nF, gsg-modules:0402, F.Cu at (135.9, 87.9)
- added C30: 18pF, gsg-modules:0402, F.Cu at (152.1, 84.6)
- added C31: 100pF, gsg-modules:0402, F.Cu at (138.7, 112.5)
- added C32: 100pF, gsg-modules:0402, F.Cu at (159.5, 102.9)
- added C33: 220nF, gsg-modules:0402, F.Cu at (136.1, 111.3)
- added C34: 220nF, gsg-modules:0402, F.Cu at (162.1, 103.4)
- added C35: 27pF, gsg-modules:0402, F.Cu at (136.1, 110.2)
- added C36: 100pF, gsg-modules:0402, F.Cu at (142.7, 111.8)
- added C37: 27pF, gsg-modules:0402, F.Cu at (162.1, 104.4)
- added C38: 100pF, gsg-modules:0402, F.Cu at (156.5, 103.6)
- added C39: 200nF, gsg-modules:0402, F.Cu at (132.3, 109.5)
- added C4: 220nF, gsg-modules:0402, F.Cu at (162.4, 79.4)
- added C40: 220nF, gsg-modules:0402, F.Cu at (144.5, 111.8)
- added C41: 220nF, gsg-modules:0402, F.Cu at (146.6, 110.7)
- added C42: 200nF, gsg-modules:0402, F.Cu at (165.6, 105.4)
- added C43: 220nF, gsg-modules:0402, F.Cu at (154.7, 103.9)
- added C44: 220nF, gsg-modules:0402, F.Cu at (152.7, 104.9)
- added C45: 27pF, gsg-modules:0402, F.Cu at (132.3, 108.5)
- added C46: 27pF, gsg-modules:0402, F.Cu at (144.5, 110.7)
- added C47: 27pF, gsg-modules:0402, F.Cu at (146.6, 109.7)
- added C48: 27pF, gsg-modules:0402, F.Cu at (165.6, 106.4)
- added C49: 27pF, gsg-modules:0402, F.Cu at (154.7, 104.9)
- added C5: 27pF, gsg-modules:0402, F.Cu at (135.9, 86.9)
- added C50: 27pF, gsg-modules:0402, F.Cu at (152.7, 105.9)
- added C51: 18pF, gsg-modules:0402, F.Cu at (146.6, 108.7)
- added C52: 18pF, gsg-modules:0402, F.Cu at (152.7, 106.9)
- added C53: 1nF, gsg-modules:0402, F.Cu at (135.6, 106.4)
- added C54: 220nF, gsg-modules:0402, F.Cu at (145.5, 102.4)
- added C55: 1nF, gsg-modules:0402, F.Cu at (163.8, 108.5)
- added C56: 220nF, gsg-modules:0402, F.Cu at (153.7, 113.0)
- added C57: 27pF, gsg-modules:0402, F.Cu at (144.5, 102.4)
- added C58: 18pF, gsg-modules:0402, F.Cu at (146.6, 107.2)
- added C59: 27pF, gsg-modules:0402, F.Cu at (154.7, 113.0)
- added C6: 100pF, gsg-modules:0402, F.Cu at (143.0, 87.4)
- added C60: 18pF, gsg-modules:0402, F.Cu at (152.7, 108.5)
- added C61: 1pF, gsg-modules:0402, F.Cu at (119.4, 91.9)
- added C62: 1pF, gsg-modules:0402, F.Cu at (120.3, 99.2)
- added C63: 1pF, gsg-modules:0402, F.Cu at (171.2, 95.2)
- added C64: 1pF, gsg-modules:0402, F.Cu at (121.9, 90.4)
- added C65: 1pF, gsg-modules:0402, F.Cu at (117.7, 100.7)
- added C66: 1pF, gsg-modules:0402, F.Cu at (169.7, 92.7)
- added C67: 10nF, gsg-modules:0402, F.Cu at (119.4, 88.9)
- added C68: 10nF, gsg-modules:0402, F.Cu at (120.4, 88.9)
- added C69: 10nF, gsg-modules:0402, F.Cu at (120.3, 102.2)
- added C7: 27pF, gsg-modules:0402, F.Cu at (162.4, 80.4)
- added C70: 10nF, gsg-modules:0402, F.Cu at (119.3, 102.2)
- added C71: 10nF, gsg-modules:0402, F.Cu at (168.1, 95.2)
- added C72: 10nF, gsg-modules:0402, F.Cu at (168.1, 94.2)
- added C73: 1pF, gsg-modules:0402, F.Cu at (115.1, 90.7)
- added C74: 1pF, gsg-modules:0402, F.Cu at (116.1, 100.3)
- added C75: 1pF, gsg-modules:0402, F.Cu at (117.6, 89.2)
- added C76: 1pF, gsg-modules:0402, F.Cu at (113.5, 101.9)
- added C77: 10nF, gsg-modules:0402, F.Cu at (115.1, 87.6)
- added C78: 10nF, gsg-modules:0402, F.Cu at (116.1, 87.6)
- added C79: 10nF, gsg-modules:0402, F.Cu at (116.1, 103.4)
- added C8: 100pF, gsg-modules:0402, F.Cu at (156.0, 79.5)
- added C80: 10nF, gsg-modules:0402, F.Cu at (115.1, 103.4)
- added C9: 200nF, gsg-modules:0402, F.Cu at (132.6, 85.9)
- added J10: TEST_2P, gsg-modules:0603-JUMPER, F.Cu at (102.1, 83.3)
- added J11: TEST_2P, gsg-modules:0603-JUMPER, F.Cu at (103.6, 115.8)
- added J12: TEST_2P, gsg-modules:0603-JUMPER, F.Cu at (103.9, 113.8)
- added J13: TEST_2P, gsg-modules:0603-JUMPER, F.Cu at (153.7, 90.9)
- added J14: TEST_2P, gsg-modules:0603-JUMPER, F.Cu at (153.7, 92.2)
- added J15: TEST_2P, gsg-modules:0603-JUMPER, F.Cu at (155.7, 114.0)
- added J16: TEST_2P, gsg-modules:0603-JUMPER, F.Cu at (157.0, 114.0)
- added J17: Conn_Coaxial, gsg-modules:SMA-EDGE, F.Cu at (177.5, 95.2)
- added J18: Conn_Coaxial, gsg-modules:SMA-EDGE, F.Cu at (109.7, 95.5)
- added J19: TEST_2P, gsg-modules:0603-JUMPER, F.Cu at (101.3, 77.7)
- added J20: TEST_2P, gsg-modules:0603-JUMPER, F.Cu at (102.1, 79.5)
- added J21: TEST_2P, gsg-modules:0603-JUMPER, F.Cu at (105.7, 106.2)
- added J22: TEST_2P, gsg-modules:0603-JUMPER, F.Cu at (106.2, 108.2)
- added J23: TEST_2P, gsg-modules:0603-JUMPER, F.Cu at (162.6, 89.2)
- added J24: TEST_2P, gsg-modules:0603-JUMPER, F.Cu at (162.6, 87.9)
- added J25: TEST_2P, gsg-modules:0603-JUMPER, F.Cu at (162.3, 113.5)
- added J26: TEST_2P, gsg-modules:0603-JUMPER, F.Cu at (162.3, 112.3)
- added J27: Conn_01x04, gsg-modules:HEADER-1x4, F.Cu at (146.8, 95.2)
- added J28: Conn_01x04, gsg-modules:HEADER-1x4, F.Cu at (158.2, 95.2)
- added J3: Conn_01x06, gsg-modules:HEADER-2x3, F.Cu at (125.2, 84.3)
- added J4: Conn_01x06, gsg-modules:HEADER-2x3, F.Cu at (173.5, 83.8)
- added J5: Conn_01x06, gsg-modules:HEADER-2x3, F.Cu at (125.2, 106.7)
- added J6: Conn_01x06, gsg-modules:HEADER-2x3, F.Cu at (173.5, 106.7)
- added J8: Conn_01x04, gsg-modules:HEADER-1x4, F.Cu at (135.4, 95.5)
- added J9: TEST_2P, gsg-modules:0603-JUMPER, F.Cu at (101.1, 84.8)
- added L1: 2n7, gsg-modules:0402, F.Cu at (120.4, 91.9)
- added L10: 2n7, gsg-modules:0402, F.Cu at (116.1, 90.7)
- added L11: 2n7, gsg-modules:0402, F.Cu at (115.1, 100.3)
- added L12: 2n7, gsg-modules:0402, F.Cu at (113.5, 89.2)
- added L13: 9n5, gsg-modules:0402, F.Cu at (115.6, 89.2)
- added L14: 2n7, gsg-modules:0402, F.Cu at (117.6, 101.9)
- added L15: 9n5, gsg-modules:0402, F.Cu at (115.6, 101.9)
- added L2: 2n7, gsg-modules:0402, F.Cu at (119.3, 99.2)
- added L3: 2n7, gsg-modules:0402, F.Cu at (171.2, 94.2)
- added L4: 2n7, gsg-modules:0402, F.Cu at (117.9, 90.4)
- added L5: 9n5, gsg-modules:0402, F.Cu at (119.9, 90.4)
- added L6: 2n7, gsg-modules:0402, F.Cu at (121.8, 100.7)
- added L7: 9n5, gsg-modules:0402, F.Cu at (119.8, 100.7)
- added L8: 2n7, gsg-modules:0402, F.Cu at (169.7, 96.8)
- added L9: 9n5, gsg-modules:0402, F.Cu at (169.7, 94.7)
- added R1: 27k, gsg-modules:0402, F.Cu at (137.4, 88.1)
- added R2: 27k, gsg-modules:0402, F.Cu at (160.8, 78.7)
- added R3: 10k, gsg-modules:0402, F.Cu at (137.2, 80.3)
- added R4: 10k, gsg-modules:0402, F.Cu at (161.5, 86.6)
- added R5: 27k, gsg-modules:0402, F.Cu at (137.7, 112.5)
- added R6: 27k, gsg-modules:0402, F.Cu at (160.5, 102.9)
- added R7: 10k, gsg-modules:0402, F.Cu at (137.7, 104.4)
- added R8: 10k, gsg-modules:0402, F.Cu at (161.8, 111.0)
- added U1: ADF7242, gsg-modules:LFCSP32, F.Cu at (140.7, 83.3)
- added U2: ADF7242, gsg-modules:LFCSP32, F.Cu at (140.7, 107.7)
- added U3: ADF7242, gsg-modules:LFCSP32, F.Cu at (158.5, 83.3)
- added U4: ADF7242, gsg-modules:LFCSP32, F.Cu at (158.5, 107.7)
- added U5: SKY13322, gsg-modules:SKY13322-375LF, F.Cu at (117.6, 95.5)
- added X1: XTAL4PIN, gsg-modules:XTAL3.2x2.5mm, F.Cu at (146.3, 81.3)
- added X2: XTAL4PIN, gsg-modules:XTAL3.2x2.5mm, F.Cu at (152.1, 86.6)
- added X3: XTAL4PIN, gsg-modules:XTAL3.2x2.5mm, F.Cu at (146.6, 104.9)
- added X4: XTAL4PIN, gsg-modules:XTAL3.2x2.5mm, F.Cu at (152.7, 110.5)
- moved J7 0.76 mm to (145.3, 76.2)
Connections:
- net /VBUS renamed Net-(J2-Pad2)
- J1 pad 10: (no net) -> /P1_1
- J1 pad 11: (no net) -> /CLK0
- J1 pad 12: (no net) -> /P1_2
- J1 pad 13: (no net) -> /P1_5
- J1 pad 14: (no net) -> /P5_2
- J1 pad 15: (no net) -> /P1_7
- J1 pad 16: (no net) -> /P1_6
- J1 pad 17: (no net) -> /P1_9
- J1 pad 18: (no net) -> /P1_8
- J1 pad 19: (no net) -> /P5_3
- J1 pad 20: (no net) -> /P1_10
- J1 pad 21: (no net) -> /P1_12
- J1 pad 22: (no net) -> /P1_11
- J1 pad 23: (no net) -> /P5_5
- J1 pad 24: (no net) -> /P5_4
- J1 pad 25: (no net) -> /P1_14
- J1 pad 26: (no net) -> /P1_13
- J1 pad 27: (no net) -> /P5_6
- J1 pad 28: (no net) -> /P1_15
- J1 pad 29: (no net) -> /P5_7
- J1 pad 3: (no net) -> /P4_9
- J1 pad 30: (no net) -> /P1_16
- J1 pad 31: (no net) -> /P1_18
- J1 pad 32: (no net) -> /P1_17
- J1 pad 33: (no net) -> /P9_5
- J1 pad 34: (no net) -> /P9_6
- J1 pad 35: (no net) -> /P2_0
- J1 pad 36: (no net) -> /P6_0
- J1 pad 37: (no net) -> /P1_20
- J1 pad 38: (no net) -> /P1_19
- J1 pad 39: (no net) -> /P1_4
- J1 pad 4: (no net) -> /P0_0
- J1 pad 40: (no net) -> /P1_3
- J1 pad 5: (no net) -> /P4_10
- J1 pad 6: (no net) -> /P0_1
- J1 pad 7: (no net) -> /P1_0
- J1 pad 8: (no net) -> /P5_0
- J1 pad 9: (no net) -> /P5_1
- J2 pad 10: (no net) -> /P4_6
- J2 pad 11: (no net) -> /P4_7
- J2 pad 12: (no net) -> /CLK2
- J2 pad 13: (no net) -> /P2_8
- J2 pad 14: (no net) -> /P2_7
- J2 pad 15: (no net) -> /P2_6
- J2 pad 16: (no net) -> /P7_7
- J2 pad 17: (no net) -> /WAKEUP0
- J2 pad 18: (no net) -> /P2_5
- J2 pad 19: (no net) -> /P2_4
- J2 pad 20: (no net) -> /P2_3
- J2 pad 21: (no net) -> /PF_4
- J2 pad 22: (no net) -> /P3_2
- J2 pad 23: (no net) -> /P7_2
- J2 pad 24: (no net) -> /P3_1
- J2 pad 25: (no net) -> /P7_1
- J2 pad 26: (no net) -> /P3_0
- J2 pad 27: (no net) -> /P7_0
- J2 pad 28: (no net) -> /P3_4
- J2 pad 29: (no net) -> /P6_8
- J2 pad 3: (no net) -> /P4_8
- J2 pad 30: (no net) -> /P3_7
- J2 pad 31: (no net) -> /P6_7
- J2 pad 32: (no net) -> /P3_3
- J2 pad 33: (no net) -> /P2_2
- J2 pad 34: (no net) -> /P6_6
- J2 pad 35: (no net) -> /P2_1
- J2 pad 36: (no net) -> /P6_3
- J2 pad 37: (no net) -> /P3_5
- J2 pad 38: (no net) -> /P3_6
- J2 pad 39: (no net) -> /I2C0_SDA
- J2 pad 4: (no net) -> /P4_0
- J2 pad 40: (no net) -> /I2C0_SCL
- J2 pad 5: (no net) -> /ADC0_0
- J2 pad 6: (no net) -> /P4_5
- J2 pad 7: (no net) -> /P4_4
- J2 pad 8: (no net) -> /P4_2
- J2 pad 9: (no net) -> /P4_3
- J7 pad 11: (no net) -> /RESET
- J7 pad 12: (no net) -> /VBAT
- J7 pad 13: (no net) -> /P2_11
- J7 pad 14: (no net) -> /P2_10
- J7 pad 15: (no net) -> /P6_10
- J7 pad 16: (no net) -> /P6_9
- J7 pad 17: (no net) -> /P6_2
- J7 pad 18: (no net) -> /P6_1
- J7 pad 2: (no net) -> /P6_4
- J7 pad 3: (no net) -> /P6_5
- J7 pad 4: (no net) -> /ADC0_5
- J7 pad 5: (no net) -> /ADC0_2
- J7 pad 6: (no net) -> /P2_9
- J7 pad 7: (no net) -> /P2_12
- J7 pad 8: (no net) -> /P2_13
- J7 pad 9: (no net) -> /RTC_ALARM
Routing:
- net GND: track 0.00 -> 121.2 mm, vias 0 -> 44
- net /P1_3: track 0.00 -> 79.2 mm, vias 0 -> 1
- net /RFOUT4_P: track 0.00 -> 68.2 mm
- net /RFOUT4_N: track 0.00 -> 67.7 mm
- net /P1_12: track 0.00 -> 58.2 mm, vias 0 -> 3
- net /P1_14: track 0.00 -> 39.7 mm, vias 0 -> 2
- net /RFOUT2_N: track 0.00 -> 38.7 mm
- net /DT4: track 0.00 -> 38.3 mm, vias 0 -> 1
- net /RFOUT2_P: track 0.00 -> 37.5 mm
- net VCC: track 0.00 -> 32.4 mm, vias 0 -> 8
- net /RFOUT1_P: track 0.00 -> 30.4 mm
- net /RFOUT1_N: track 0.00 -> 29.5 mm
- net /IRQ1: track 0.00 -> 28.7 mm, vias 0 -> 1
- net /DT3: track 0.00 -> 27.7 mm
- net /P1_13: track 0.00 -> 26.0 mm, vias 0 -> 1
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Other:
- board text added: "16 July 2018"
- board text added: "GreatFET Lucky Bamboo"
- board text added: "RX"
- board text added: "TX"
- board text removed: "27 September 2015"
- board text removed: "GreatFET Neighbor"
