File: azalea/azalea.sch (KiCad schematic (older format))
At the start: 103 parts, among them J1 NEIGHBOR1, J2 NEIGHBOR2, J3 USB-MICRO-B-SHIELDED, J4 USB-MICRO-B-SHIELDED, J5 JTAG, J6 POWER, J7 BONUS_ROW, SW1 DFU, SW2 RESET, U1 LPC4330FBD144, U2 W25Q16DV, U3 AP7333, U4 IP4220CZ6, U5 AP2553W6-7, X1 MCU_XTAL, X2 RTC_XTAL

Commit message: Azalea: do not populate 32 kHz oscillator (X2, C1, and C2).
Parts:
- C1, C2, X2: Note (none) -> DNP
Other:
- note added: "You may populate the 32 kHz\ncrystal oscillator (X2, C1, and C2)\nfor RTC operation, but the\nrecommended alternative is to\nsupply an external 32 kHz signal\non RTCX1 (J7 pin 10). See the\nLPC4330 errata."
Changed lines of the file:
@@
 F 5 "C0603C180J5GAC" H 2000 8900 60  0001 C CNN "Part Number"
 F 6 "CAP CER 18PF 50V 5% NP0 0603" H 2000 8900 60  0001 C CNN "Description"
+F 7 "DNP" H 2250 8900 60  0000 C CNN "Note"
 	1    2000 8900
 	1    0    0    -1
@@
 F 5 "C0603C180J5GAC" H 1500 8900 60  0001 C CNN "Part Number"
 F 6 "CAP CER 18PF 50V 5% NP0 0603" H 1500 8900 60  0001 C CNN "Description"
+F 7 "DNP" H 1250 8900 60  0000 C CNN "Note"
 	1    1500 8900
 	1    0    0    -1
@@
 F 5 "AB26TRQ-32.768KHZ-T" H 1750 8550 60  0001 C CNN "Part Number"
 F 6 "CRYSTAL 32.768KHZ 12.5PF SMD" H 1750 8550 60  0001 C CNN "Description"
+F 7 "DNP" H 1750 8800 60  0000 C CNN "Note"
 	1    1750 8550
 	1    0    0    -1
@@
 Text Label 15150 7550 1    40   ~ 0
 RTCX1
+Text Notes 1050 10200 0    60   ~ 0
+You may populate the 32 kHz\ncrystal oscillator (X2, C1, and C2)\nfor RTC operation, but the\nrecommended alternative is to\nsupply an external 32 kHz signal\non RTCX1 (J7 pin 10).  See the\nLPC4330 errata.
 $EndSCHEMATC
