File: luckybamboo/luckybamboo.sch (KiCad schematic (older format))
At the start: 148 parts, among them J1 NEIGHBOR1, J10 TEST_2P, J11 TEST_2P, J12 TEST_2P, J13 TEST_2P, J14 TEST_2P, J15 TEST_2P, J16 TEST_2P, J17 Conn_Coaxial, J18 Conn_Coaxial, J19 TEST_2P, J2 NEIGHBOR2, J20 TEST_2P, J21 TEST_2P, J22 TEST_2P, J23 TEST_2P, J24 TEST_2P, J25 TEST_2P, J26 TEST_2P, J27 TEST_2P, J28 TEST_2P, J29 TEST_2P, J3 Conn_01x08, J30 TEST_2P, J31 TEST_2P, J32 TEST_2P, J33 TEST_2P, J4 Conn_01x08, J5 Conn_01x08, J6 Conn_01x08, J7 BONUS_ROW, J8 TEST_2P, J9 TEST_2P, U1 ADF7242, U10 ADF7242_balun, U11 ADF7242_balun, U14 ADF7242_balun, U15 ADF7242_balun, U16 ADF7242_balun, U17 ADF7242_balun, U2 ADF7242, U3 ADF7242, U4 ADF7242, U5 SKY13322, U8 ADF7242_balun, U9 ADF7242_balun, X1 XTAL4PIN, X2 XTAL4PIN, X3 XTAL4PIN, X4 XTAL4PIN

Commit message: renamed Orchid to Lucky Bamboo
Parts:
- C1, C10, C11, C12, C13, C14, C15, C16, C17, C18, C19, C2, C20, C21, C22, C23, C24, C25, C26, C27, C28, C29, C3, C30, C31, C32, C33, C34, C35, C36, C37, C38, C39, C4, C40, C41, C42, C43, C44, C45, C46, C47, C48, C49, C5, C50, C51, C52, C53, C54, C55, C56, C57, C58, C59, C6, C60, C63, C64, C65, C68, C69, C7, C70, C71, C72, C73, C74, C75, C76, C77, C78, C79, C8, C80, C81, C9: symbol orchid-rescue:C -> luckybamboo-rescue:C
- J1, J2: symbol orchid-rescue:CONN_02X20 -> luckybamboo-rescue:CONN_02X20
- J10, J11, J12, J13, J14, J15, J16, J19, J20, J21, J22, J23, J24, J25, J26, J27, J28, J29, J30, J31, J32, J33, J8, J9: symbol orchid-rescue:TEST_2P -> luckybamboo-rescue:TEST_2P
- J17, J18: symbol orchid-rescue:Conn_Coaxial -> luckybamboo-rescue:Conn_Coaxial
- J3, J4, J5, J6: symbol orchid-rescue:Conn_01x08 -> luckybamboo-rescue:Conn_01x08
- J7: symbol orchid-rescue:Conn_01x20 -> luckybamboo-rescue:Conn_01x20
- L1: symbol orchid-rescue:L -> luckybamboo-rescue:L
- MH1, MH2, MH3, MH4: symbol orchid-rescue:Conn_01x01 -> luckybamboo-rescue:Conn_01x01
- R1, R2, R3, R4, R5, R6, R7, R8: symbol orchid-rescue:R -> luckybamboo-rescue:R
- U1, U2, U3, U4: symbol orchid-rescue:ADF7242 -> luckybamboo-rescue:ADF7242
- U10, U11, U14, U15, U16, U17, U8, U9: symbol orchid-rescue:ADF7242_balun -> luckybamboo-rescue:ADF7242_balun
- U5: symbol orchid-rescue:SKY13322 -> luckybamboo-rescue:SKY13322
- X1, X2, X3, X4: symbol orchid-rescue:XTAL4PIN -> luckybamboo-rescue:XTAL4PIN

Commit message: Completed new amplifier/splitter section in schematic and layout.
Parts:
- C61: renamed from C?; symbol RF_divider_test-rescue:C -> luckybamboo-rescue:C; Description (none) -> CAP CER 1000PF 10V X7R 0402; Manufacturer (none) -> Wurth Electronics Inc.; Part Number (none) -> 885012205006
- R10, R11, R9: renamed from R?; footprint gsg-modules:0603 -> gsg-modules:0402; symbol RF_divider_test-rescue:R -> luckybamboo-rescue:R; Description (none) -> RES 100 OHM 5% 1/16W 0402; Manufacturer (none) -> Stackpole Electronics Inc.; Part Number (none) -> RMCF0402JT100R
- U12, U6, U7: renamed from U?; symbol RF_divider_test-rescue:HHM2293A1 -> gsg-symbols:HHM2293A1; Description (none) -> MULTILAYER DIVIDER FOR W-LAN/BLU; Manufacturer (none) -> TDK Corporation; Part Number (none) -> HHM2293A1
- U13: renamed from U?; footprint gsg-modules:TSNP-6-2 -> gsg-modules:BGA7H1N6; symbol RF_divider_test-rescue:BGA7H1N6 -> gsg-symbols:BGA7H1N6; Description (none) -> IC AMP LTE 2.3-2.69GHZ TSNP6-2; Manufacturer (none) -> Infineon Technologies; Part Number (none) -> BGA7H1N6E6327XTSA1
Connections:
- no-connect marks 57 -> 61
Other:
- moved on the sheet: R10, R9
