File: foxglove/power_supplies.sch (KiCad schematic (older format))
At the start: 10 parts

Commit message: Added multiplexors to bank A
Parts:
- removed C? (x2): 0.1uF, symbol Device:C
- removed R?: 10k, symbol Device:R
- removed U?: BH2226FV, symbol gsg-symbols:BH2226FV
- removed U? (x2): MC4558CPT, symbol gsg-symbols:MC4558CPT
- added C? (x2): 10uF, symbol Device:C
- added C? (x2): 0.47uF, symbol Device:C
- added J?: Conn_01x02_Female, symbol Connector:Conn_01x02_Female
- added R?: 10k, symbol Device:R
- added U?: DAC084S085, symbol gsg-symbols:DAC084S085
- added U? (x2): MIC94310, symbol gsg-symbols:MIC94310
Connections:
- net labels added: +1V2, +2V5, DAC2, DAC3, DAC4
- net labels removed: High_thr, Low_thr, MISO, MOSI, SCK
- wire segments 93 -> 68
Other:
- note added: "1.2V and 2.5V\nvoltage regulators"
- note added: "optional external \nsupply input"
- note removed: "DAC output: 0-5V"
- note removed: "DAC, SPI interface"
- moved on the sheet: C?, U?
