File: foxglove/shifters.sch (KiCad schematic (older format))
At the start: 20 parts

Commit message: Added multiplexors to bank A
Parts:
- removed C? (x4): 0.1uF, symbol Device:C
- removed J?: RJ45, gsg-modules:RJ45-RJHSE-5380, symbol Connector:RJ45_Shielded
- removed P?: CONN_02X05, gsg-modules:HEADER-2x5, symbol Connector_Generic:Conn_02x05_Odd_Even
- removed U?: SHIFTER0, gsg-modules:SOT363, symbol gsg-symbols:74LVC1T45
- removed U?: SHIFTER1, gsg-modules:SOT363, symbol gsg-symbols:74LVC1T45
- removed U?: SHIFTER2, gsg-modules:SOT363, symbol gsg-symbols:74LVC1T45
- removed U?: SHIFTER4, gsg-modules:SOT363, symbol gsg-symbols:74LVC1T45
- removed U?: SHIFTER5, gsg-modules:SOT363, symbol gsg-symbols:74LVC1T45
- removed U?: SHIFTER6, gsg-modules:SOT363, symbol gsg-symbols:74LVC1T45
- removed U?: SHIFTER7, gsg-modules:SOT363, symbol gsg-symbols:74LVC1T45
- removed U?: SHIFTER3, gsg-modules:SOT363, symbol gsg-symbols:74LVC1T45
- removed U?: NCD9830, symbol gsg-symbols:NCD9830
- removed U? (x3): LM339, symbol gsg-symbols:LM339
- added J? (x2): Conn_02x05_Odd_Even, symbol Connector_Generic:Conn_02x05_Odd_Even
- added R? (x16): R, symbol Device:R
- added R?: 5k, symbol Device:R
- added R?: 10k, symbol Device:R
- added U? (x8): 74HC4051, symbol 74xx:74HC4051
- added U?: SHIFTER1, gsg-modules:SOT363, symbol gsg-symbols:74LVC1T45
- added U?: SHIFTER2, gsg-modules:SOT363, symbol gsg-symbols:74LVC1T45
- added U?: SHIFTER3, gsg-modules:SOT363, symbol gsg-symbols:74LVC1T45
- added U?: SHIFTER4, gsg-modules:SOT363, symbol gsg-symbols:74LVC1T45
- added U?: SHIFTER5, gsg-modules:SOT363, symbol gsg-symbols:74LVC1T45
- added U?: SHIFTER6, gsg-modules:SOT363, symbol gsg-symbols:74LVC1T45
- added U?: SHIFTER7, gsg-modules:SOT363, symbol gsg-symbols:74LVC1T45
- added U?: SHIFTER8, gsg-modules:SOT363, symbol gsg-symbols:74LVC1T45
Connections:
- net labels added: +1V2, A1_shift, A2_shift, A3_shift, A4_shift, A5_shift, A6_shift, A7_shift, A8, A8_shift, ADC, B8, COMP1, COMP2, COMP_O1, COMP_O2, COMP_O3, COMP_O4, DAC2, DAC3, DAC4, DIR8, gf_adc
- net labels removed: A0, A0_high, A0_low, A1_high, A1_low, A2_high, A2_low, A3_high, A3_low, A4_high, A4_low, A5_high, A5_low, A6_high, A6_low, A7_high, A7_low, B0, DIR0, High_thr, Low_thr
- wire segments 132 -> 141
- no-connect marks 1 -> 0
Other:
- note added: "bank A: ADC, DAC, level shifter, pull-up, pull-down, comparator\nbank B: FPGA"
- note added: "comparator bank"
- note added: "voltage divider to keep signal\nwithin 3.3V ADC range"
- note removed: "0<Vthr<VCC-2"
- note removed: "1.2 < VCC < 5.5"
- note removed: "ADC, I2C interface"
- moved on the sheet: C?, U?
