File: neighbor-template/neighbor-template.sch (KiCad schematic (older format))
At the start: 7 parts, among them J1 NEIGHBOR1, J2 NEIGHBOR2, J7 BONUS_ROW

Commit message: Updates to jasmine schematic and layout; Updated neighbor-template to be compatible with KiCAD 5.1.2
Parts:
- added JP? (x3): Jumper_3_Bridged12, symbol Jumper:Jumper_3_Bridged12
- added R?: 10k, symbol Device:R
- added U?: M24C02-FMN6TP, Package_SO:SOIC-8_3.9x4.9mm_P1.27mm, symbol Memory_EEPROM:M24C02-FMN
- J1, J2: symbol CONN_02X20 -> Connector_Generic:Conn_02x20_Odd_Even
- J7: symbol CONN_01X20 -> Connector_Generic:Conn_01x20; Note DNP -> (none)
- MH1, MH2, MH3, MH4: symbol CONN_01X01 -> Connector_Generic:Conn_01x01
Connections:
- net GND: now also JP?.1 (A), JP?.1 (A), JP?.1 (A), U?.4 (VSS)
- net I2C0_SCL: now also U?.6 (SCL)
- net I2C0_SDA: now also U?.5 (SDA)
- net P2_1: now also R?.1, U?.7 (~WC)
- net VBUS: now also J2.2 (Pin_2)
- net VCC: now also JP?.3 (B), JP?.3 (B), JP?.3 (B), R?.2, U?.8 (VCC)
- new net: JP?.2 (C), U?.1 (E0)
- new net: JP?.2 (C), U?.2 (E1)
- new net: JP?.2 (C), U?.3 (E2)
Other:
- note added: "WC is by default pulled up, and the write protection is locked.\nTo enable write configuration ... FIXME"
